Commit message: Prepared Gripper

File: code/ros/minibot_moveit_config/config/minibot.srdf.xacro (robot description, xacro)
@@ -1,7 +1,3 @@
 <?xml version='1.0' encoding='utf-8'?>
-<!--This does not replace URDF, and is not an extension of URDF.
-    This is a format for representing semantic information about the robot structure.
-    A URDF file must exist for this robot as well, where the joints and the links that are referenced are defined
--->
 <robot xmlns:xacro="http://www.ros.org/wiki/xacro" name="minibot">
     <!--GROUPS: Representation of a set of joints and links. This can be useful for specifying DOF to plan for, defining arms, end effectors, etc-->
@@ -32,5 +28,34 @@
       <link name="finger_right_link" />
     </group>
+    <group name="minibot_gripper">
+      <link name="knuckle_link" />
+      <link name="knuckle_left_link" />
+      <link name="knuckle_right_link" />
+      <link name="finger_link" />
+      <link name="finger_centre_link" />
+      <link name="finger_left_link" />
+      <link name="finger_right_link" />
+    </group>
+    <group name="minibot">
+      <link name="base_link" />
+      <link name="shoulder_link" />
+      <link name="upperarm_link" />
+      <link name="elbow_link" />
+      <link name="forearm_link" />
+      <link name="wrist_link" />
+      <link name="flange_link" />
+      <link name="tool0_link" />
+      <link name="knuckle_link" />
+      <link name="knuckle_left_link" />
+      <link name="knuckle_right_link" />
+      <link name="finger_link" />
+      <link name="finger_centre_link" />
+      <link name="finger_left_link" />
+      <link name="finger_right_link" />
+    </group>
     <!--GROUP STATES: Purpose: Define a named state for a particular group, in terms of joint values. This is useful to define states like 'folded arms'-->
+    <!--      -->
+    <!-- arm  -->
+    <!--      -->
     <group_state name="ready_for_action" group="minibot_arm">
       <joint name="base_joint" value="0" />
@@ -49,15 +74,46 @@
       <joint name="wrist_joint" value="0" />
     </group_state>
-    <group_state name="pinching" group="palm">
-      <joint name="knuckle_joint" value="1.04" />
+    <!--         -->
+    <!-- gripper -->
+    <!--         -->
+    <group_state name="pinching" group="minibot_gripper">
+      <joint name="knuckle_joint" value="0" />
+      <joint name="palm_left_joint" value="0" />
+      <joint name="palm_right_joint" value="0" />
+      <joint name="finger_joint" value="0" />
+      <joint name="finger_centre_joint" value="0" />
+      <joint name="finger_left_joint" value="0" />
     </group_state>
-    <group_state name="gripping" group="palm">
+    <group_state name="seamonster" group="minibot_gripper">
       <joint name="knuckle_joint" value="0" />
+      <joint name="palm_left_joint" value="0" />
+      <joint name="palm_right_joint" value="0" />
+      <joint name="finger_joint" value="0" />
+      <joint name="finger_right_joint" value="0" />
+      <joint name="finger_left_joint" value="0" />
     </group_state>
-    <group_state name="open" group="hand">
-      <joint name="finger_joint" value="1.04" />
+    <group_state name="snake" group="minibot_gripper">
+      <joint name="knuckle_joint" value="0" />
+      <joint name="palm_left_joint" value="0" />
+      <joint name="palm_right_joint" value="0" />
+      <joint name="finger_joint" value="0" />
+      <joint name="finger_right_joint" value="0" />
+      <joint name="finger_left_joint" value="0" />
     </group_state>
-    <group_state name="tight" group="hand">
+    <group_state name="egggrip" group="minibot_gripper">
+      <joint name="knuckle_joint" value="0" />
+      <joint name="palm_left_joint" value="0" />
+      <joint name="palm_right_joint" value="0" />
       <joint name="finger_joint" value="0" />
+      <joint name="finger_right_joint" value="0" />
+      <joint name="finger_left_joint" value="0" />
+    </group_state>
+    <group_state name="gripping" group="minibot_gripper">
+      <joint name="knuckle_joint" value="0" />
+      <joint name="palm_left_joint" value="0" />
+      <joint name="palm_right_joint" value="0" />
+      <joint name="finger_joint" value="0" />
+      <joint name="finger_right_joint" value="0" />
+      <joint name="finger_left_joint" value="0" />
     </group_state>
     <!--VIRTUAL JOINT: Purpose: this element defines a virtual joint between a robot link and an external frame of reference (considered fixed with respect to the robot)-->

File: code/ros/minibot_moveit_config/config/minibot.urdf (robot description, URDF)
Before this commit: robot minibot, 16 links, 15 joints
Links:
- link base_link: geometry collision mesh filename=package://minibot_moveit_config/config/stl/base_collision.s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; visual mesh filename=package://minibot_moveit_config/config/stl/base.stl
- link elbow_link: geometry collision mesh filename=package://minibot_moveit_config/config/stl/elbow_collision.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; visual mesh filename=package://minibot_moveit_config/config/stl/elbow.stl
- link finger_centre_link: geometry collision mesh filename=package://minibot_moveit_config/config/stl/finger_collision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; visual mesh filename=package://minibot_moveit_config/config/stl/finger.stl
- link finger_left_link: geometry collision mesh filename=package://minibot_moveit_config/config/stl/finger_collision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; visual mesh filename=package://minibot_moveit_config/config/stl/finger.stl
- link finger_right_link: geometry collision mesh filename=package://minibot_moveit_config/config/stl/finger_collision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; visual mesh filename=package://minibot_moveit_config/config/stl/finger.stl
- link forearm_link: geometry collision mesh filename=package://minibot_moveit_config/config/stl/forearm_collisio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; visual mesh filename=package://minibot_moveit_config/config/stl/forearm.stl
- link knuckle_left_link: geometry visual mesh filename=package://minibot_moveit_config/config/stl/knuckle_left.stl
- link knuckle_right_link: geometry visual mesh filename=package://minibot_moveit_config/config/stl/knuckle_right.stl
- link palm_link: geometry collision mesh filename=package://minibot_moveit_config/config/stl/palm_collision.s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; visual mesh filename=package://minibot_moveit_config/config/stl/palm.stl
- link shoulder_link: geometry collision mesh filename=package://minibot_moveit_config/config/stl/shoulder_collisi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; visual mesh filename=package://minibot_moveit_config/config/stl/shoulder.stl
- link upperarm_link: geometry collision mesh filename=package://minibot_moveit_config/config/stl/upperarm_collisi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; visual mesh filename=package://minibot_moveit_config/config/stl/upperarm.stl
- link wrist_link: geometry visual mesh filename=package://minibot_moveit_config/config/stl/wrist.stl

Commit message: prepared for ODROID

File: code/ros/minibot_moveit_config/config/minibot.srdf.xacro (robot description, xacro)
@@ -30,11 +30,13 @@
     <group name="minibot_gripper">
       <link name="knuckle_link" />
-      <link name="knuckle_left_link" />
-      <link name="knuckle_right_link" />
+      <!-- <link name="knuckle_left_link" />-->
+      <!--<link name="knuckle_right_link" />-->
       <link name="finger_link" />
-      <link name="finger_centre_link" />
+      <!--<link name="finger_centre_link" />
       <link name="finger_left_link" />
       <link name="finger_right_link" />
+    -->
     </group>
+    <end_effector name="gripper" group="minibot_gripper" parent_link="flange_link" parent_group="minibot_arm"/>
     <group name="minibot">
       <link name="base_link" />
@@ -46,11 +48,11 @@
       <link name="flange_link" />
       <link name="tool0_link" />
-      <link name="knuckle_link" />
-      <link name="knuckle_left_link" />
-      <link name="knuckle_right_link" />
+      <link  name="knuckle_link" />
+      <!-- <link name="knuckle_left_link" />-->
+      <!--<link name="knuckle_right_link" />-->
       <link name="finger_link" />
-      <link name="finger_centre_link" />
-      <link name="finger_left_link" />
-      <link name="finger_right_link" />
+      <!--<link name="finger_centre_link" />-->
+      <!--<link name="finger_left_link" />-->
+      <!--<link name="finger_right_link" />-->
     </group>
     <!--GROUP STATES: Purpose: Define a named state for a particular group, in terms of joint values. This is useful to define states like 'folded arms'-->
@@ -79,41 +81,21 @@
     <group_state name="pinching" group="minibot_gripper">
       <joint name="knuckle_joint" value="0" />
-      <joint name="palm_left_joint" value="0" />
-      <joint name="palm_right_joint" value="0" />
       <joint name="finger_joint" value="0" />
-      <joint name="finger_centre_joint" value="0" />
-      <joint name="finger_left_joint" value="0" />
     </group_state>
     <group_state name="seamonster" group="minibot_gripper">
       <joint name="knuckle_joint" value="0" />
-      <joint name="palm_left_joint" value="0" />
-      <joint name="palm_right_joint" value="0" />
       <joint name="finger_joint" value="0" />
-      <joint name="finger_right_joint" value="0" />
-      <joint name="finger_left_joint" value="0" />
     </group_state>
     <group_state name="snake" group="minibot_gripper">
       <joint name="knuckle_joint" value="0" />
-      <joint name="palm_left_joint" value="0" />
-      <joint name="palm_right_joint" value="0" />
       <joint name="finger_joint" value="0" />
-      <joint name="finger_right_joint" value="0" />
-      <joint name="finger_left_joint" value="0" />
     </group_state>
     <group_state name="egggrip" group="minibot_gripper">
       <joint name="knuckle_joint" value="0" />
-      <joint name="palm_left_joint" value="0" />
-      <joint name="palm_right_joint" value="0" />
       <joint name="finger_joint" value="0" />
-      <joint name="finger_right_joint" value="0" />
-      <joint name="finger_left_joint" value="0" />
     </group_state>
     <group_state name="gripping" group="minibot_gripper">
       <joint name="knuckle_joint" value="0" />
-      <joint name="palm_left_joint" value="0" />
-      <joint name="palm_right_joint" value="0" />
       <joint name="finger_joint" value="0" />
-      <joint name="finger_right_joint" value="0" />
-      <joint name="finger_left_joint" value="0" />
     </group_state>
     <!--VIRTUAL JOINT: Purpose: this element defines a virtual joint between a robot link and an external frame of reference (considered fixed with respect to the robot)-->

Commit message: integrated gripper  in movement

File: code/ros/minibot_moveit_config/config/minibot.srdf.xacro (robot description, xacro)
@@ -30,11 +30,5 @@
     <group name="minibot_gripper">
       <link name="knuckle_link" />
-      <!-- <link name="knuckle_left_link" />-->
-      <!--<link name="knuckle_right_link" />-->
       <link name="finger_link" />
-      <!--<link name="finger_centre_link" />
-      <link name="finger_left_link" />
-      <link name="finger_right_link" />
-    -->
     </group>
     <end_effector name="gripper" group="minibot_gripper" parent_link="flange_link" parent_group="minibot_arm"/>
@@ -49,10 +43,5 @@
       <link name="tool0_link" />
       <link  name="knuckle_link" />
-      <!-- <link name="knuckle_left_link" />-->
-      <!--<link name="knuckle_right_link" />-->
       <link name="finger_link" />
-      <!--<link name="finger_centre_link" />-->
-      <!--<link name="finger_left_link" />-->
-      <!--<link name="finger_right_link" />-->
     </group>
     <!--GROUP STATES: Purpose: Define a named state for a particular group, in terms of joint values. This is useful to define states like 'folded arms'-->

File: code/ros/minibot_moveit_config/config/minibot.urdf (robot description, URDF)
Before this commit: robot minibot, 16 links, 15 joints
Joints:
- joint finger_joint: limit lower=-0.174532925199 upper=1.0471975512 effort=5.0 velocity=3.14159265359 -> lower=-0.174532925199 upper=1.0471975512 effort=50.0 velocity=31.4159265359

File: code/ros/minibot_moveit_config/config/minibot.urdf.xacro (robot description, xacro)
@@ -254,5 +254,5 @@
      <child link="finger_link"/>
      <axis xyz="0 1 0" />
-     <limit effort="5.0" lower="${-10/180*pi}" upper="${60/180*pi}" velocity="${180/180*pi}" />
+     <limit effort="50.0" lower="${-10/180*pi}" upper="${60/180*pi}" velocity="${1800/180*pi}" />
   </joint>
   <link name="finger_link">

Commit message: regenerated IKfast with 7 digits precision

File: code/ros/minibot_moveit_config/config/minibot.srdf.xacro (robot description, xacro)
@@ -15,5 +15,4 @@
       <link name="flange_link" />
       <link name="tool0_link" />
-      <!-- <chain base_link="base_link" tip_link="tool0_link" /> -->
     </group>
     <group name="palm">

File: code/ros/minibot_moveit_config/config/minibot.urdf (robot description, URDF)
Before this commit: robot minibot, 16 links, 15 joints
Joints:
- joint tool0_joint: origin xyz=0 0 0.10 rpy=0 0 0 -> xyz=0 0 0.0 rpy=0 0 0

File: code/ros/minibot_moveit_config/config/minibot.urdf.xacro (robot description, xacro)
@@ -7,5 +7,4 @@
   <xacro:property name="palm_color" value="${214/255} ${195/255} ${59/255} 1.0"/>
   <xacro:property name="finger_color" value="0.62 0.25 0.25 1.0"/>
-  <xacro:property name="wrist2tcp" value="0.10"/>
   <link name="base_link">
     <visual>
@@ -163,5 +162,5 @@
   <!--  ####################### -->
   <joint name="tool0_joint" type="fixed">
-     <origin rpy="0 0 0"  xyz="0 0 0.10"/>
+     <origin rpy="0 0 0"  xyz="0 0 0.0"/>
      <parent link="flange_link"/>
      <child link="tool0_link"/>
