Commit message: 75mm tool difference

File: code/ros/minibot_moveit_config/config/minibot.urdf.xacro (robot description, xacro)
@@ -162,5 +162,5 @@
   <!--  ####################### -->
   <joint name="tool0_joint" type="fixed">
-     <origin rpy="0 0 0"  xyz="0 0 0.0"/>
+     <origin rpy="0 0 0"  xyz="0 0 0.075"/>
      <parent link="flange_link"/>
      <child link="tool0_link"/>
